File: Hardware/SparkX_EZ_Header.brd (EAGLE design)
At the start: 10.7 x 40.6 mm, 48 parts, among them J1 QWIIC_RIGHT_ANGLE

Commit message: Add bottom silk
Parts:
- added LOGO3: OSHW-LOGOMINI, SparkFun-Aesthetics:OSHW-LOGO-MINI
- added LOGO4: QWIIC_LOGO_5MM, SparkFun-Aesthetics:QWIIC_5MM
- added U$20: SPARKX-LOGO3, SparkX:SPARKX-SMALL
- added U$22: (no value), output:#V_USB#0
- added U$23, U$24: (no value), output:#3#3V#0
- added U$25: (no value), output:#PWR_EN#0
- added U$26, U$27: (no value), output:#GND#0
- added U$28: (no value), output:#SCLK#0
- added U$29: (no value), output:#COPI#0
- added U$30: (no value), output:#SDA#0
- added U$31: (no value), output:#CIPO#0
- added U$32: (no value), output:#GPIO1#0
- added U$33: (no value), output:#CS0#0
- added U$34: (no value), output:#GPIO0#0
- added U$35: (no value), output:#CS1#0
- added U$36: (no value), output:#CS2#0
- added U$37: (no value), output:EZ_HEADER0
- added U$38: (no value), output:#SCL#0
Changed lines of the file:
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@@
 <element name="U$21" library="output" package="EZ_HEADER0" value="" x="5.334" y="8.255" smashed="yes"/>
 <element name="U$9" library="output" package="#SCL#0" value="" x="3.8735" y="20.7645" smashed="yes"/>
+<element name="U$20" library="SparkX" package="SPARKX-SMALL" value="SPARKX-LOGO3" x="5.334" y="7.62" smashed="yes" rot="MR0"/>
+<element name="U$22" library="output" package="#V_USB#0" value="" x="4.5085" y="13.208" smashed="yes" rot="MR0"/>
+<element name="U$23" library="output" package="#3#3V#0" value="" x="3.937" y="15.6845" smashed="yes" rot="MR0"/>
+<element name="U$24" library="output" package="#3#3V#0" value="" x="6.731" y="14.7955" smashed="yes" rot="MR0"/>
+<element name="U$25" library="output" package="#PWR_EN#0" value="" x="5.6515" y="12.192" smashed="yes" rot="MR0"/>
+<element name="U$26" library="output" package="#GND#0" value="" x="6.731" y="17.3355" smashed="yes" rot="MR0"/>
+<element name="U$27" library="output" package="#GND#0" value="" x="4.0005" y="18.2245" smashed="yes" rot="MR0"/>
+<element name="U$28" library="output" package="#SCLK#0" value="" x="6.477" y="19.8755" smashed="yes" rot="MR0"/>
+<element name="U$29" library="output" package="#COPI#0" value="" x="6.604" y="22.4155" smashed="yes" rot="MR0"/>
+<element name="U$30" library="output" package="#SDA#0" value="" x="3.937" y="23.3045" smashed="yes" rot="MR0"/>
+<element name="U$31" library="output" package="#CIPO#0" value="" x="6.604" y="24.892" smashed="yes" rot="MR0"/>
+<element name="U$32" library="output" package="#GPIO1#0" value="" x="4.318" y="25.8445" smashed="yes" rot="MR0"/>
+<element name="U$33" library="output" package="#CS0#0" value="" x="6.7945" y="27.432" smashed="yes" rot="MR0"/>
+<element name="U$34" library="output" package="#GPIO0#0" value="" x="4.3815" y="28.448" smashed="yes" rot="MR0"/>
+<element name="U$35" library="output" package="#CS1#0" value="" x="6.858" y="30.0355" smashed="yes" rot="MR0"/>
+<element name="U$36" library="output" package="#CS2#0" value="" x="3.8735" y="30.9245" smashed="yes" rot="MR0"/>
+<element name="U$37" library="output" package="EZ_HEADER0" value="" x="5.334" y="5.715" smashed="yes" rot="MR0"/>
+<element name="U$38" library="output" package="#SCL#0" value="" x="3.8735" y="20.7645" smashed="yes" rot="MR0"/>
+<element name="LOGO3" library="SparkFun-Aesthetics" package="OSHW-LOGO-MINI" value="OSHW-LOGOMINI" x="5.334" y="3.175" smashed="yes" rot="MR0"/>
+<element name="LOGO4" library="SparkFun-Aesthetics" package="QWIIC_5MM" value="QWIIC_LOGO_5MM" x="5.334" y="39.37" smashed="yes" rot="MR0"/>
 </elements>
 <signals>

Commit message: Gapless production panel
Other:
- board text added: "2-Layer Board 1.6mm Thickness 1oz Copper (Outer layers) HASL Finish"
- board text removed: "2-Layer Board 1.6mm Thickness 1oz Copper (Outer layers) HASL Finish When running the panelizer, add a vertical gap of 0.2" to make the boards easier to separate"
Changed lines of the file:
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@@
 <layer number="23" name="tOrigins" color="15" fill="1" visible="yes" active="yes"/>
 <layer number="24" name="bOrigins" color="15" fill="1" visible="yes" active="yes"/>
-<layer number="25" name="tNames" color="57" fill="1" visible="yes" active="yes"/>
-<layer number="26" name="bNames" color="57" fill="1" visible="yes" active="yes"/>
-<layer number="27" name="tValues" color="7" fill="1" visible="yes" active="yes"/>
-<layer number="28" name="bValues" color="7" fill="1" visible="yes" active="yes"/>
-<layer number="29" name="tStop" color="7" fill="3" visible="yes" active="yes"/>
-<layer number="30" name="bStop" color="7" fill="6" visible="yes" active="yes"/>
-<layer number="31" name="tCream" color="7" fill="4" visible="yes" active="yes"/>
-<layer number="32" name="bCream" color="7" fill="5" visible="yes" active="yes"/>
-<layer number="33" name="tFinish" color="6" fill="3" visible="yes" active="yes"/>
-<layer number="34" name="bFinish" color="6" fill="6" visible="yes" active="yes"/>
-<layer number="35" name="tGlue" color="7" fill="4" visible="yes" active="yes"/>
-<layer number="36" name="bGlue" color="7" fill="5" visible="yes" active="yes"/>
-<layer number="37" name="tTest" color="7" fill="1" visible="yes" active="yes"/>
-<layer number="38" name="bTest" color="7" fill="1" visible="yes" active="yes"/>
-<layer number="39" name="tKeepout" color="4" fill="11" visible="yes" active="yes"/>
-<layer number="40" name="bKeepout" color="1" fill="11" visible="yes" active="yes"/>
-<layer number="41" name="tRestrict" color="4" fill="10" visible="yes" active="yes"/>
-<layer number="42" name="bRestrict" color="1" fill="10" visible="yes" active="yes"/>
-<layer number="43" name="vRestrict" color="2" fill="10" visible="yes" active="yes"/>
-<layer number="44" name="Drills" color="7" fill="1" visible="yes" active="yes"/>
+<layer number="25" name="tNames" color="57" fill="1" visible="no" active="yes"/>
+<layer number="26" name="bNames" color="57" fill="1" visible="no" active="yes"/>
+<layer number="27" name="tValues" color="7" fill="1" visible="no" active="yes"/>
+<layer number="28" name="bValues" color="7" fill="1" visible="no" active="yes"/>
+<layer number="29" name="tStop" color="7" fill="3" visible="no" active="yes"/>
+<layer number="30" name="bStop" color="7" fill="6" visible="no" active="yes"/>
+<layer number="31" name="tCream" color="7" fill="4" visible="no" active="yes"/>
+<layer number="32" name="bCream" color="7" fill="5" visible="no" active="yes"/>
+<layer number="33" name="tFinish" color="6" fill="3" visible="no" active="yes"/>
+<layer number="34" name="bFinish" color="6" fill="6" visible="no" active="yes"/>
+<layer number="35" name="tGlue" color="7" fill="4" visible="no" active="yes"/>
+<layer number="36" name="bGlue" color="7" fill="5" visible="no" active="yes"/>
+<layer number="37" name="tTest" color="7" fill="1" visible="no" active="yes"/>
+<layer number="38" name="bTest" color="7" fill="1" visible="no" active="yes"/>
+<layer number="39" name="tKeepout" color="4" fill="11" visible="no" active="yes"/>
+<layer number="40" name="bKeepout" color="1" fill="11" visible="no" active="yes"/>
+<layer number="41" name="tRestrict" color="4" fill="10" visible="no" active="yes"/>
+<layer number="42" name="bRestrict" color="1" fill="10" visible="no" active="yes"/>
+<layer number="43" name="vRestrict" color="2" fill="10" visible="no" active="yes"/>
+<layer number="44" name="Drills" color="7" fill="1" visible="no" active="yes"/>
 <layer number="45" name="Holes" color="7" fill="1" visible="yes" active="yes"/>
-<layer number="46" name="Milling" color="3" fill="1" visible="yes" active="yes"/>
-<layer number="47" name="Measures" color="7" fill="1" visible="yes" active="yes"/>
-<layer number="48" name="Document" color="7" fill="1" visible="yes" active="yes"/>
-<layer number="49" name="Reference" color="7" fill="1" visible="yes" active="yes"/>
-<layer number="50" name="dxf" color="7" fill="1" visible="yes" active="yes"/>
+<layer number="46" name="Milling" color="3" fill="1" visible="no" active="yes"/>
+<layer number="47" name="Measures" color="7" fill="1" visible="no" active="yes"/>
+<layer number="48" name="Document" color="7" fill="1" visible="no" active="yes"/>
+<layer number="49" name="Reference" color="7" fill="1" visible="no" active="yes"/>
+<layer number="50" name="dxf" color="7" fill="1" visible="no" active="yes"/>
 <layer number="51" name="tDocu" color="6" fill="1" visible="yes" active="yes"/>
-<layer number="52" name="bDocu" color="7" fill="1" visible="yes" active="yes"/>
+<layer number="52" name="bDocu" color="7" fill="1" visible="no" active="yes"/>
 <layer number="2" name="Route2" color="63" fill="1" visible="no" active="no"/>
 <layer number="15" name="Route15" color="23" fill="1" visible="no" active="no"/>
@@
 1oz Copper (Outer layers)
 HASL Finish
-When running the panelizer, add a vertical gap of 0.2"
-to make the boards easier to separate</text>
+</text>
 <dimension x1="0" y1="0" x2="10.668" y2="0" x3="5.334" y3="-3.81" textsize="1.778" textratio="15" layer="47" dtype="horizontal" unit="inch"/>
 <dimension x1="0" y1="40.64" x2="0" y2="0" x3="-6.350003125" y3="20.32" textsize="1.778" textratio="15" layer="47" dtype="vertical" unit="inch"/>

Commit message: Update 16-way FPC Connector
Parts:
- OUT: value FPC_16_0.5MM_BACKFLIP -> (none); device New_Parts_Connectors:FPC_16_DOUBLESIDED_BACKFLIP -> SparkFun-Connectors:FPC_16_0.5MM
Changed lines of the file:
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@@
 <element name="FD3" library="SparkFun-Aesthetics" package="FIDUCIAL-MICRO" value="FIDUCIALUFIDUCIAL" x="10.033" y="0.635" smashed="yes"/>
 <element name="FD4" library="SparkFun-Aesthetics" package="FIDUCIAL-MICRO" value="FIDUCIALUFIDUCIAL" x="10.033" y="0.635" smashed="yes" rot="MR0"/>
-<element name="OUT" library="New_Parts_Connectors" package="FPC_16_DOUBLESIDED_BACKFLIP" value="FPC_16_0.5MM_BACKFLIP" x="5.334" y="2.0955" smashed="yes" rot="R180">
-<attribute name="ATOM_PART" value="FPC05016-42201" x="5.334" y="2.0955" size="1.778" layer="27" font="vector" ratio="15" rot="R180" display="off"/>
-<attribute name="PROD_ID" value="" x="5.334" y="2.0955" size="1.778" layer="27" font="vector" ratio="15" rot="R180" display="off"/>
+<element name="OUT" library="SparkFun-Connectors" package="FPC_16_0.5MM" value="" x="5.334" y="2.0955" smashed="yes" rot="R180">
+<attribute name="PROD_ID" value="CONN-16066" x="5.334" y="2.0955" size="1.778" layer="27" font="vector" ratio="15" rot="R180" display="off"/>
 </element>
 <element name="LOGO2" library="SparkFun-Aesthetics" package="OSHW-LOGO-MINI" value="OSHW-LOGOMINI" x="1.651" y="32.5755" smashed="yes"/>
