File: Hardware/Production/SparkX_smol_Header-Panel.brd (EAGLE design)
At the start: 198.4 x 137.2 mm, 3174 parts, among them J1 QWIIC_RIGHT_ANGLE, J10 QWIIC_RIGHT_ANGLE, J11 QWIIC_RIGHT_ANGLE, J12 QWIIC_RIGHT_ANGLE, J13 QWIIC_RIGHT_ANGLE, J14 QWIIC_RIGHT_ANGLE, J15 QWIIC_RIGHT_ANGLE, J16 QWIIC_RIGHT_ANGLE, J17 QWIIC_RIGHT_ANGLE, J18 QWIIC_RIGHT_ANGLE, J19 QWIIC_RIGHT_ANGLE, J2 QWIIC_RIGHT_ANGLE, J20 QWIIC_RIGHT_ANGLE, J21 QWIIC_RIGHT_ANGLE, J22 QWIIC_RIGHT_ANGLE, J23 QWIIC_RIGHT_ANGLE, J24 QWIIC_RIGHT_ANGLE, J25 QWIIC_RIGHT_ANGLE, J26 QWIIC_RIGHT_ANGLE, J27 QWIIC_RIGHT_ANGLE, J28 QWIIC_RIGHT_ANGLE, J29 QWIIC_RIGHT_ANGLE, J3 QWIIC_RIGHT_ANGLE, J30 QWIIC_RIGHT_ANGLE, J31 QWIIC_RIGHT_ANGLE, J32 QWIIC_RIGHT_ANGLE, J33 QWIIC_RIGHT_ANGLE, J34 QWIIC_RIGHT_ANGLE, J35 QWIIC_RIGHT_ANGLE, J36 QWIIC_RIGHT_ANGLE, J37 QWIIC_RIGHT_ANGLE, J38 QWIIC_RIGHT_ANGLE, J39 QWIIC_RIGHT_ANGLE, J4 QWIIC_RIGHT_ANGLE, J40 QWIIC_RIGHT_ANGLE, J41 QWIIC_RIGHT_ANGLE, J42 QWIIC_RIGHT_ANGLE, J43 QWIIC_RIGHT_ANGLE, J44 QWIIC_RIGHT_ANGLE, J45 QWIIC_RIGHT_ANGLE, J46 QWIIC_RIGHT_ANGLE, J47 QWIIC_RIGHT_ANGLE, J48 QWIIC_RIGHT_ANGLE, J5 QWIIC_RIGHT_ANGLE, J6 QWIIC_RIGHT_ANGLE, J7 QWIIC_RIGHT_ANGLE, J8 QWIIC_RIGHT_ANGLE, J9 QWIIC_RIGHT_ANGLE

Commit message: Update smôl logo
Parts:
- added U$1825, U$1846, U$1864: (no value), output:#CS0#0
- added U$1826, U$1847, U$1865: (no value), output:#GPIO0#0
- added U$1827, U$1848, U$1866: (no value), output:#CS1#0
- added U$1828, U$1849, U$1867: (no value), output:#CS2#0
- added U$1829, U$1851, U$1868: (no value), output:#SCL#0
- added U$1830, U$1831, U$1869, U$1870: (no value), output:SM�L_HEADER0
- added U$1832, U$1871: (no value), output:OUT0
- added U$1833, U$1872: SMOL_LOGOSMALL, SparkX:SMOL_SMALL
- added U$1834, U$1852: SPARKX-LOGO3, SparkX:SPARKX-SMALL
- added U$1835, U$1853: (no value), output:#V_USB#0
- added U$1836, U$1837, U$1854, U$1855: (no value), output:#3#3V#0
- added U$1838, U$1856: (no value), output:#PWR_EN#0
- added U$1839, U$1840, U$1857, U$1858: (no value), output:#GND#0
- added U$1841, U$1859: (no value), output:#SCLK#0
- added U$1842, U$1860: (no value), output:#COPI#0
- added U$1843, U$1861: (no value), output:#SDA#0
- added U$1844, U$1862: (no value), output:#CIPO#0
- added U$1845, U$1863: (no value), output:#GPIO1#0
- added U$1850: (no value), output:#I�C#0
- U$100, U$120, U$121, U$138, U$139, U$1564, U$1582, U$159, U$1602, U$1603, U$1620, U$1621, U$1641, U$1659, U$177, U$784, U$82, U$822, U$823, U$861, U$880, U$918, U$919, U$957: device output:#GND#0 -> output:#3#3V#0
- U$1000, U$1038, U$1684, U$1702, U$1722, U$1740, U$202, U$220, U$240, U$258, U$904, U$942: device output:#GPIO1#0 -> output:#GND#0
- U$1001, U$1685, U$1703, U$203, U$221, U$905: device output:#CS0#0 -> output:#SCLK#0
- U$1002, U$1686, U$1704, U$204, U$222, U$906: device output:#GPIO0#0 -> output:#COPI#0
- U$1003, U$1687, U$1705, U$205, U$223, U$907: device output:#CS1#0 -> output:#SDA#0
- U$1004, U$1688, U$1706, U$206, U$224, U$908: device output:#CS2#0 -> output:#CIPO#0
- U$1005, U$1689, U$207: device output:#I�C#0 -> output:#GPIO1#0
- U$1006, U$1669, U$1690, U$187, U$208, U$871: device output:#SCL#0 -> output:#CS0#0
- U$1007, U$1691, U$1787, U$209, U$305, U$989: value SPARKX-LOGO3 -> (none); device SparkX:SPARKX-SMALL -> output:#GPIO0#0
- U$1008, U$1692, U$1788, U$210, U$306, U$990: device output:#V_USB#0 -> output:#CS1#0
- U$1009, U$1030, U$1048, U$1693, U$1732, U$1789, U$211, U$250, U$307, U$346, U$991: device output:#3#3V#0 -> output:#CS2#0
- U$101, U$1526, U$1544, U$1565, U$1583, U$44, U$62, U$746, U$785, U$83, U$842, U$881: device output:#GND#0 -> output:#PWR_EN#0
- U$1010, U$135, U$1617, U$1656, U$174, U$1751, U$1790, U$269, U$308, U$915, U$954, U$971: device output:#3#3V#0 -> output:#SCL#0
- U$1011, U$1753, U$1791, U$271, U$309, U$973: device output:#PWR_EN#0 -> output:SM�L_HEADER0
- U$1012, U$1050, U$1051, U$1089, U$1792, U$310, U$348, U$349, U$387: device output:#GND#0 -> output:SM�L_HEADER0
- U$1013, U$1754, U$1793, U$272, U$311, U$974: device output:#GND#0 -> output:OUT0
- U$1014, U$1794, U$312: value (none) -> SMOL_LOGOSMALL; device output:#SCLK#0 -> SparkX:SMOL_SMALL
- U$1015, U$1111, U$1795, U$1813, U$313, U$331: value (none) -> SPARKX-LOGO3; device output:#COPI#0 -> SparkX:SPARKX-SMALL
- U$1016, U$1112, U$1796, U$1814, U$314, U$332: device output:#SDA#0 -> output:#V_USB#0
- U$1017, U$1075, U$1113, U$1759, U$1777, U$1797, U$1815, U$277, U$295, U$315, U$333, U$979: device output:#CIPO#0 -> output:#3#3V#0
- U$1018, U$1056, U$1114, U$1152, U$1798, U$1816, U$316, U$334, U$354, U$372: device output:#GPIO1#0 -> output:#3#3V#0
- U$1019, U$1115, U$1799, U$1817, U$317, U$335: device output:#CS0#0 -> output:#PWR_EN#0
- U$102, U$1528, U$1546, U$1566, U$1584, U$46, U$64, U$748, U$786, U$84, U$844, U$882: device output:#SCLK#0 -> output:#GND#0
- U$1020, U$1078, U$1116, U$1762, U$1780, U$1800, U$1818, U$280, U$298, U$318, U$336, U$982: device output:#GPIO0#0 -> output:#GND#0
- U$1021, U$1059, U$1117, U$1155, U$1801, U$1819, U$319, U$337, U$357, U$375: device output:#CS1#0 -> output:#GND#0
- U$1022, U$1118, U$1802, U$1820, U$320, U$338: device output:#CS2#0 -> output:#SCLK#0
- U$1023, U$1158, U$1821, U$339, U$360: device output:#SCL#0 -> output:#COPI#0
- U$1024, U$1063, U$1822, U$340, U$379: device output:SM�L_HEADER0 -> output:#SDA#0
- U$1025, U$1784, U$1823, U$302, U$341, U$986: device output:SM�L_HEADER0 -> output:#CIPO#0
- U$1026, U$1824, U$342: device output:OUT0 -> output:#GPIO1#0
- U$1027, U$1045, U$1729, U$247, U$343: value SPARKX-LOGO3 -> (none); device SparkX:SPARKX-SMALL -> output:#CS0#0
- U$1028, U$1046, U$1730, U$248, U$344: device output:#V_USB#0 -> output:#GPIO0#0
- U$1029, U$1047, U$1068, U$1086, U$1731, U$1770, U$249, U$288, U$345, U$384: device output:#3#3V#0 -> output:#CS1#0
- U$103, U$123, U$141, U$1567, U$1585, U$1605, U$1623, U$787, U$825, U$85, U$883, U$921: device output:#COPI#0 -> output:#GND#0
- U$1031, U$1733, U$251: device output:#PWR_EN#0 -> output:#I�C#0
- U$1032, U$1071, U$1088, U$1127, U$1734, U$1773, U$252, U$291, U$386, U$425: device output:#GND#0 -> output:#SCL#0
- U$1033, U$1678, U$1696, U$1717, U$1735, U$196, U$214, U$235, U$253, U$898, U$937, U$994: value (none) -> SPARKX-LOGO3; device output:#GND#0 -> SparkX:SPARKX-SMALL
- U$1034, U$1718, U$1736, U$236, U$254, U$938: device output:#SCLK#0 -> output:#V_USB#0
- U$1035, U$1681, U$1699, U$1719, U$1737, U$199, U$217, U$237, U$255, U$901, U$939, U$997: device output:#COPI#0 -> output:#3#3V#0
- U$1036, U$1074, U$1720, U$1738, U$1758, U$1776, U$238, U$256, U$276, U$294, U$940, U$978: device output:#SDA#0 -> output:#3#3V#0
- U$1037, U$1721, U$1739, U$239, U$257, U$941: device output:#CIPO#0 -> output:#PWR_EN#0
- U$1039, U$1077, U$1723, U$1741, U$1761, U$1779, U$241, U$259, U$279, U$297, U$943, U$981: device output:#CS0#0 -> output:#GND#0
- U$104, U$1568, U$1586, U$788, U$86, U$884: device output:#SDA#0 -> output:#SCLK#0
- U$1040, U$1724, U$1742, U$242, U$260, U$944: device output:#GPIO0#0 -> output:#SCLK#0
- U$1041, U$1725, U$1743, U$243, U$261, U$945: device output:#CS1#0 -> output:#COPI#0
- U$1042, U$1726, U$1744, U$244, U$262, U$946: device output:#CS2#0 -> output:#SDA#0
- U$1043, U$1727, U$245: device output:#I�C#0 -> output:#CIPO#0
- U$1044, U$1707, U$1728, U$225, U$246, U$909: device output:#SCL#0 -> output:#GPIO1#0
- U$1049, U$1695, U$213, U$347, U$993: device output:#PWR_EN#0 -> output:#SCL#0
- U$105, U$1569, U$1587, U$789, U$87, U$885: device output:#CIPO#0 -> output:#COPI#0
- U$1052, U$350: device output:#SCLK#0 -> output:OUT0
- U$1053, U$351: value (none) -> SMOL_LOGOSMALL; device output:#COPI#0 -> SparkX:SMOL_SMALL
- U$1054, U$1150, U$352, U$370: value (none) -> SPARKX-LOGO3; device output:#SDA#0 -> SparkX:SPARKX-SMALL
- U$1055, U$1151, U$353, U$371: device output:#CIPO#0 -> output:#V_USB#0
- U$1057, U$1095, U$1153, U$1191, U$355, U$373, U$393, U$411: device output:#CS0#0 -> output:#3#3V#0
- U$1058, U$1154, U$356, U$374: device output:#GPIO0#0 -> output:#PWR_EN#0
- U$106, U$1570, U$1588, U$790, U$88, U$886: device output:#GPIO1#0 -> output:#SDA#0
- U$1060, U$1098, U$1156, U$1194, U$358, U$376, U$396, U$414: device output:#CS2#0 -> output:#GND#0
- U$1061, U$1196, U$377, U$398: device output:#SCL#0 -> output:#SCLK#0
- U$1062, U$1101, U$378, U$417: device output:SM�L_HEADER0 -> output:#COPI#0
- U$1064, U$380: device output:OUT0 -> output:#CIPO#0
- U$1065, U$1083, U$1767, U$285, U$381: value SPARKX-LOGO3 -> (none); device SparkX:SPARKX-SMALL -> output:#GPIO1#0
- U$1066, U$1084, U$1768, U$286, U$382: device output:#V_USB#0 -> output:#CS0#0
- U$1067, U$1085, U$1106, U$1124, U$1769, U$1808, U$287, U$326, U$383, U$422: device output:#3#3V#0 -> output:#GPIO0#0
- U$1069, U$1087, U$1771, U$289, U$385: device output:#PWR_EN#0 -> output:#CS2#0
- U$107, U$1571, U$1589, U$791, U$887, U$89: device output:#CS0#0 -> output:#CIPO#0
- U$1070, U$1109, U$1772, U$1811, U$290, U$329: device output:#GND#0 -> output:#I�C#0
- U$1072, U$1756, U$1774, U$274, U$292, U$976: value (none) -> SPARKX-LOGO3; device output:#SCLK#0 -> SparkX:SPARKX-SMALL
- U$1073, U$1757, U$1775, U$275, U$293, U$977: device output:#COPI#0 -> output:#V_USB#0
- U$1076, U$1760, U$1778, U$278, U$296, U$980: device output:#GPIO1#0 -> output:#PWR_EN#0
- U$1079, U$1763, U$1781, U$281, U$299, U$983: device output:#CS1#0 -> output:#SCLK#0
- U$108, U$1572, U$1590, U$792, U$888, U$90: device output:#GPIO0#0 -> output:#GPIO1#0
- U$1080, U$1764, U$1782, U$282, U$300, U$984: device output:#CS2#0 -> output:#COPI#0
- U$1081, U$1765, U$283: device output:#I�C#0 -> output:#SDA#0
- U$1082, U$1745, U$1766, U$263, U$284, U$947: device output:#SCL#0 -> output:#CIPO#0
- U$109, U$1573, U$1591, U$793, U$889, U$91: device output:#CS1#0 -> output:#CS0#0
- U$1090, U$1128, U$388, U$426: device output:#SCLK#0 -> output:SM�L_HEADER0
- U$1091, U$389: device output:#COPI#0 -> output:OUT0
- U$1092, U$390: value (none) -> SMOL_LOGOSMALL; device output:#SDA#0 -> SparkX:SMOL_SMALL
- U$1093, U$1189, U$391, U$409: value (none) -> SPARKX-LOGO3; device output:#CIPO#0 -> SparkX:SPARKX-SMALL
- U$1094, U$1190, U$392, U$410: device output:#GPIO1#0 -> output:#V_USB#0
- U$1096, U$1134, U$1192, U$1230, U$394, U$412, U$432, U$450: device output:#GPIO0#0 -> output:#3#3V#0
- U$1097, U$1193, U$395, U$413: device output:#CS1#0 -> output:#PWR_EN#0
- U$1099, U$1137, U$1234, U$1272, U$415, U$436, U$453, U$474: device output:#SCL#0 -> output:#GND#0
- U$110, U$1574, U$1592, U$794, U$890, U$92: device output:#CS2#0 -> output:#GPIO0#0
- U$1100, U$1139, U$416, U$455: device output:SM�L_HEADER0 -> output:#SCLK#0
- U$1102, U$418: device output:OUT0 -> output:#SDA#0
- U$1103, U$1121, U$1805, U$323, U$419: value SPARKX-LOGO3 -> (none); device SparkX:SPARKX-SMALL -> output:#CIPO#0
- U$1104, U$1122, U$1806, U$324, U$420: device output:#V_USB#0 -> output:#GPIO1#0
- U$1105, U$1123, U$1144, U$1162, U$1807, U$325, U$364, U$421, U$460: device output:#3#3V#0 -> output:#CS0#0
- U$1107, U$1125, U$1809, U$327, U$423: device output:#PWR_EN#0 -> output:#CS1#0
- U$1108, U$1126, U$1147, U$1165, U$1810, U$328, U$367, U$424, U$463: device output:#GND#0 -> output:#CS2#0
- U$111, U$132, U$1593, U$1614, U$795, U$930: device output:#SCL#0 -> output:#CS1#0
- U$1110, U$1166, U$1812, U$330, U$464: device output:#SCLK#0 -> output:#SCL#0
- U$1119, U$1803, U$321: device output:#I�C#0 -> output:#COPI#0
- U$112, U$151, U$1594, U$1633, U$796, U$835: device output:SM�L_HEADER0 -> output:#CS2#0
- U$1120, U$1783, U$1804, U$301, U$322, U$985: device output:#SCL#0 -> output:#SDA#0
- U$1129, U$1167, U$427, U$465: device output:#COPI#0 -> output:SM�L_HEADER0
- U$113, U$1556, U$1595, U$720, U$74, U$759: device output:SM�L_HEADER0 -> output:#SCL#0
- U$1130, U$428: device output:#SDA#0 -> output:OUT0
- U$1131, U$429: value (none) -> SMOL_LOGOSMALL; device output:#CIPO#0 -> SparkX:SMOL_SMALL
- U$1132, U$1228, U$430, U$448: value (none) -> SPARKX-LOGO3; device output:#GPIO1#0 -> SparkX:SPARKX-SMALL
- U$1133, U$1229, U$431, U$449: device output:#CS0#0 -> output:#V_USB#0
- U$1135, U$1173, U$1231, U$1269, U$433, U$451, U$471, U$489: device output:#CS1#0 -> output:#3#3V#0
- U$1136, U$1232, U$434, U$452: device output:#CS2#0 -> output:#PWR_EN#0
- U$1138, U$1176, U$1177, U$1215, U$454, U$492, U$493, U$531: device output:SM�L_HEADER0 -> output:#GND#0
- U$114, U$1558, U$1596, U$76: device output:OUT0 -> output:SM�L_HEADER0
- U$1140, U$456: device output:OUT0 -> output:#COPI#0
- U$1141, U$1159, U$361, U$457: value SPARKX-LOGO3 -> (none); device SparkX:SPARKX-SMALL -> output:#SDA#0
- U$1142, U$1160, U$362, U$458: device output:#V_USB#0 -> output:#CIPO#0
- U$1143, U$1161, U$1182, U$1200, U$363, U$402, U$459, U$498: device output:#3#3V#0 -> output:#GPIO1#0
- U$1145, U$1163, U$365, U$461: device output:#PWR_EN#0 -> output:#GPIO0#0
- U$1146, U$1164, U$1185, U$1203, U$366, U$405, U$462, U$501: device output:#GND#0 -> output:#CS1#0
- U$1148, U$368: device output:#SCLK#0 -> output:#I�C#0
- U$1149, U$1205, U$369, U$503: device output:#COPI#0 -> output:#SCL#0
- U$115, U$153, U$1597, U$1635, U$817, U$855: value SPARKX-LOGO3 -> (none); device SparkX:SPARKX-SMALL -> output:SM�L_HEADER0
- U$1157, U$359: device output:#I�C#0 -> output:#SCLK#0
- U$116, U$1598, U$818: device output:#V_USB#0 -> output:OUT0
- U$1168, U$1206, U$466, U$504: device output:#SDA#0 -> output:SM�L_HEADER0
- U$1169, U$467: device output:#CIPO#0 -> output:OUT0
- U$117, U$156, U$1599, U$1638, U$819, U$858: value (none) -> SMOL_LOGOSMALL; device output:#3#3V#0 -> SparkX:SMOL_SMALL
- U$1170, U$468: value (none) -> SMOL_LOGOSMALL; device output:#GPIO1#0 -> SparkX:SMOL_SMALL
- U$1171, U$1267, U$469, U$487: value (none) -> SPARKX-LOGO3; device output:#CS0#0 -> SparkX:SPARKX-SMALL
- U$1172, U$1268, U$470, U$488: device output:#GPIO0#0 -> output:#V_USB#0
- U$1174, U$1212, U$1270, U$1308, U$472, U$490, U$510, U$528: device output:#CS2#0 -> output:#3#3V#0
- U$1175, U$1310, U$491, U$512: device output:#SCL#0 -> output:#PWR_EN#0
- U$1178, U$494: device output:OUT0 -> output:#SCLK#0
- U$1179, U$1197, U$399, U$495: value SPARKX-LOGO3 -> (none); device SparkX:SPARKX-SMALL -> output:#COPI#0
- U$118, U$136, U$1561, U$1579, U$1600, U$1618, U$781, U$79, U$820, U$877, U$916, U$97: value (none) -> SPARKX-LOGO3; device output:#3#3V#0 -> SparkX:SPARKX-SMALL
- U$1180, U$1198, U$400, U$496: device output:#V_USB#0 -> output:#SDA#0
- U$1181, U$1199, U$1220, U$1238, U$401, U$440, U$497, U$536: device output:#3#3V#0 -> output:#CIPO#0
- U$1183, U$1201, U$403, U$499: device output:#PWR_EN#0 -> output:#CS0#0
- U$1184, U$1202, U$1223, U$1241, U$404, U$443, U$500, U$539: device output:#GND#0 -> output:#GPIO0#0
- U$1186, U$1204, U$406, U$502: device output:#SCLK#0 -> output:#CS2#0
- U$1187, U$407: device output:#COPI#0 -> output:#I�C#0
- U$1188, U$1244, U$408, U$542: device output:#SDA#0 -> output:#SCL#0
- U$119, U$137, U$1601, U$1619, U$821, U$917: device output:#PWR_EN#0 -> output:#V_USB#0
- U$1195, U$1233, U$397, U$435: device output:#I�C#0 -> output:#GND#0
- U$1207, U$1245, U$505, U$543: device output:#CIPO#0 -> output:SM�L_HEADER0
- U$1208, U$506: device output:#GPIO1#0 -> output:OUT0
- U$1209, U$507: value (none) -> SMOL_LOGOSMALL; device output:#CS0#0 -> SparkX:SMOL_SMALL
- U$1210, U$1306, U$508, U$526: value (none) -> SPARKX-LOGO3; device output:#GPIO0#0 -> SparkX:SPARKX-SMALL
- U$1211, U$1307, U$509, U$527: device output:#CS1#0 -> output:#V_USB#0
- U$1213, U$1251, U$1348, U$1386, U$529, U$550, U$567, U$588: device output:#SCL#0 -> output:#3#3V#0
- U$1214, U$1253, U$530, U$569: device output:SM�L_HEADER0 -> output:#PWR_EN#0
- U$1216, U$1254, U$532, U$570: device output:OUT0 -> output:#GND#0
- U$1217, U$1235, U$437, U$533: value SPARKX-LOGO3 -> (none); device SparkX:SPARKX-SMALL -> output:#SCLK#0
- U$1218, U$1236, U$438, U$534: device output:#V_USB#0 -> output:#COPI#0
- U$1219, U$1237, U$1258, U$1276, U$439, U$478, U$535, U$574: device output:#3#3V#0 -> output:#SDA#0
- U$122, U$140, U$1604, U$1622, U$824, U$920: device output:#SCLK#0 -> output:#PWR_EN#0
- U$1221, U$1239, U$441, U$537: device output:#PWR_EN#0 -> output:#GPIO1#0
- U$1222, U$1240, U$1261, U$1279, U$442, U$481, U$538, U$577: device output:#GND#0 -> output:#CS0#0
- U$1224, U$1242, U$444, U$540: device output:#SCLK#0 -> output:#CS1#0
- U$1225, U$1243, U$445, U$541: device output:#COPI#0 -> output:#CS2#0
- U$1226, U$446: device output:#SDA#0 -> output:#I�C#0
- U$1227, U$1283, U$447, U$581: device output:#CIPO#0 -> output:#SCL#0
- U$124, U$142, U$1606, U$162, U$1624, U$1644, U$1662, U$180, U$826, U$864, U$922, U$960: device output:#SDA#0 -> output:#GND#0
- U$1246, U$1284, U$544, U$582: device output:#GPIO1#0 -> output:SM�L_HEADER0
- U$1247, U$545: device output:#CS0#0 -> output:OUT0
- U$1248, U$546: value (none) -> SMOL_LOGOSMALL; device output:#GPIO0#0 -> SparkX:SMOL_SMALL
- U$1249, U$1345, U$547, U$565: value (none) -> SPARKX-LOGO3; device output:#CS1#0 -> SparkX:SPARKX-SMALL
- U$125, U$143, U$1607, U$1625, U$827, U$923: device output:#CIPO#0 -> output:#SCLK#0
- U$1250, U$1346, U$548, U$566: device output:#CS2#0 -> output:#V_USB#0
- U$1252, U$1290, U$1291, U$1329, U$568, U$606, U$607, U$645: device output:SM�L_HEADER0 -> output:#3#3V#0
- U$1255, U$1273, U$1293, U$1311, U$475, U$513, U$571, U$609: value SPARKX-LOGO3 -> (none); device SparkX:SPARKX-SMALL -> output:#GND#0
- U$1256, U$1274, U$476, U$572: device output:#V_USB#0 -> output:#SCLK#0
- U$1257, U$1275, U$1296, U$1314, U$477, U$516, U$573, U$612: device output:#3#3V#0 -> output:#COPI#0
- U$1259, U$1277, U$479, U$575: device output:#PWR_EN#0 -> output:#CIPO#0
- U$126, U$144, U$1608, U$1626, U$828, U$924: device output:#GPIO1#0 -> output:#COPI#0
- U$1260, U$1278, U$1299, U$1317, U$480, U$519, U$576, U$615: device output:#GND#0 -> output:#GPIO1#0
- U$1262, U$1280, U$482, U$578: device output:#SCLK#0 -> output:#GPIO0#0
- U$1263, U$1281, U$483, U$579: device output:#COPI#0 -> output:#CS1#0
- U$1264, U$1282, U$484, U$580: device output:#SDA#0 -> output:#CS2#0
- U$1265, U$485: device output:#CIPO#0 -> output:#I�C#0
- U$1266, U$1322, U$486, U$620: device output:#GPIO1#0 -> output:#SCL#0
- U$127, U$145, U$1609, U$1627, U$829, U$925: device output:#CS0#0 -> output:#SDA#0
- U$1271, U$473: device output:#I�C#0 -> output:#PWR_EN#0
- U$128, U$146, U$1610, U$1628, U$830, U$926: device output:#GPIO0#0 -> output:#CIPO#0
- U$1285, U$1323, U$583, U$621: device output:#CS0#0 -> output:SM�L_HEADER0
- U$1286, U$584: device output:#GPIO0#0 -> output:OUT0
- U$1287, U$585: value (none) -> SMOL_LOGOSMALL; device output:#CS1#0 -> SparkX:SMOL_SMALL
- U$1288, U$1384, U$586, U$604: value (none) -> SPARKX-LOGO3; device output:#CS2#0 -> SparkX:SPARKX-SMALL
- U$1289, U$1424, U$605, U$626: device output:#SCL#0 -> output:#V_USB#0
- U$129, U$147, U$1611, U$1629, U$831, U$927: device output:#CS1#0 -> output:#GPIO1#0
- U$1292, U$608: device output:OUT0 -> output:#PWR_EN#0
- U$1294, U$1312, U$1332, U$1350, U$514, U$552, U$610, U$648: device output:#V_USB#0 -> output:#GND#0
- U$1295, U$1313, U$1334, U$1352, U$515, U$554, U$611, U$650: device output:#3#3V#0 -> output:#SCLK#0
- U$1297, U$1315, U$517, U$613: device output:#PWR_EN#0 -> output:#SDA#0
- U$1298, U$1316, U$1337, U$1355, U$518, U$557, U$614, U$653: device output:#GND#0 -> output:#CIPO#0
- U$130, U$148, U$1612, U$1630, U$832, U$928: device output:#CS2#0 -> output:#CS0#0
- U$1300, U$1318, U$520, U$616: device output:#SCLK#0 -> output:#CS0#0
- U$1301, U$1319, U$521, U$617: device output:#COPI#0 -> output:#GPIO0#0
- U$1302, U$1320, U$522, U$618: device output:#SDA#0 -> output:#CS1#0
- U$1303, U$1321, U$523, U$619: device output:#CIPO#0 -> output:#CS2#0
- U$1304, U$524: device output:#GPIO1#0 -> output:#I�C#0
- U$1305, U$1361, U$525, U$659: device output:#CS0#0 -> output:#SCL#0
- U$1309, U$1347, U$511, U$549: device output:#I�C#0 -> output:#3#3V#0
- U$131, U$1613, U$929: device output:#I�C#0 -> output:#GPIO0#0
- U$1324, U$1362, U$622, U$660: device output:#GPIO0#0 -> output:SM�L_HEADER0
- U$1325, U$623: device output:#CS1#0 -> output:OUT0
- U$1326, U$624: value (none) -> SMOL_LOGOSMALL; device output:#CS2#0 -> SparkX:SMOL_SMALL
- U$1327, U$1462, U$643, U$664: value (none) -> SPARKX-LOGO3; device output:#SCL#0 -> SparkX:SPARKX-SMALL
- U$1328, U$1367, U$644, U$683: device output:SM�L_HEADER0 -> output:#V_USB#0
- U$133, U$1615, U$1711, U$229, U$913, U$931: value SPARKX-LOGO3 -> (none); device SparkX:SPARKX-SMALL -> output:#CS2#0
- U$1330, U$1368, U$646, U$684: device output:OUT0 -> output:#3#3V#0
- U$1331, U$1349, U$551, U$647: value SPARKX-LOGO3 -> (none); device SparkX:SPARKX-SMALL -> output:#PWR_EN#0
- U$1333, U$1351, U$1371, U$1372, U$1389, U$1390, U$1410, U$1428, U$553, U$591, U$592, U$630, U$649, U$687, U$688, U$726: device output:#3#3V#0 -> output:#GND#0
- U$1335, U$1353, U$555, U$651: device output:#PWR_EN#0 -> output:#COPI#0
- U$1336, U$1354, U$1375, U$1393, U$556, U$595, U$652, U$691: device output:#GND#0 -> output:#SDA#0
- U$1338, U$1356, U$558, U$654: device output:#SCLK#0 -> output:#GPIO1#0
- U$1339, U$1357, U$559, U$655: device output:#COPI#0 -> output:#CS0#0
- U$134, U$1616, U$914: device output:#V_USB#0 -> output:#I�C#0
- U$1340, U$1358, U$560, U$656: device output:#SDA#0 -> output:#GPIO0#0
- U$1341, U$1359, U$561, U$657: device output:#CIPO#0 -> output:#CS1#0
- U$1342, U$1360, U$562, U$658: device output:#GPIO1#0 -> output:#CS2#0
- U$1343, U$563: device output:#CS0#0 -> output:#I�C#0
- U$1344, U$1400, U$564, U$698: device output:#GPIO0#0 -> output:#SCL#0
- U$1363, U$1401, U$661, U$699: device output:#CS1#0 -> output:SM�L_HEADER0
- U$1364, U$662: device output:#CS2#0 -> output:OUT0
- U$1365, U$702: value (none) -> SMOL_LOGOSMALL; device output:#SCL#0 -> SparkX:SMOL_SMALL
- U$1366, U$1405, U$682, U$721: value (none) -> SPARKX-LOGO3; device output:SM�L_HEADER0 -> SparkX:SPARKX-SMALL
- U$1369, U$1387, U$1407, U$1425, U$589, U$627, U$685, U$723: value SPARKX-LOGO3 -> (none); device SparkX:SPARKX-SMALL -> output:#3#3V#0
- U$1370, U$1388, U$590, U$686: device output:#V_USB#0 -> output:#PWR_EN#0
- U$1373, U$1391, U$593, U$689: device output:#PWR_EN#0 -> output:#SCLK#0
- U$1374, U$1392, U$1413, U$1431, U$594, U$633, U$690, U$729: device output:#GND#0 -> output:#COPI#0
- U$1376, U$1394, U$596, U$692: device output:#SCLK#0 -> output:#CIPO#0
- U$1377, U$1395, U$597, U$693: device output:#COPI#0 -> output:#GPIO1#0
- U$1378, U$1396, U$598, U$694: device output:#SDA#0 -> output:#CS0#0
- U$1379, U$1397, U$599, U$695: device output:#CIPO#0 -> output:#GPIO0#0
- U$1380, U$1398, U$600, U$696: device output:#GPIO1#0 -> output:#CS1#0
- U$1381, U$1399, U$601, U$697: device output:#CS0#0 -> output:#CS2#0
- U$1382, U$602: device output:#GPIO0#0 -> output:#I�C#0
- U$1383, U$1439, U$603, U$737: device output:#CS1#0 -> output:#SCL#0
- U$1385, U$587: device output:#I�C#0 -> output:#V_USB#0
- U$1402, U$1440, U$700, U$738: device output:#CS2#0 -> output:SM�L_HEADER0
- U$1403, U$740: device output:#SCL#0 -> output:OUT0
- U$1404, U$1443: value (none) -> SMOL_LOGOSMALL; device output:SM�L_HEADER0 -> SparkX:SMOL_SMALL
- U$1406, U$722: device output:OUT0 -> output:#V_USB#0
- U$1408, U$1426, U$1446, U$1464, U$628, U$666, U$724, U$762: device output:#V_USB#0 -> output:#3#3V#0
- U$1409, U$1427, U$1448, U$1466, U$629, U$668, U$725, U$764: device output:#3#3V#0 -> output:#PWR_EN#0
- U$1411, U$1429, U$1449, U$1467, U$631, U$669, U$727, U$765: device output:#PWR_EN#0 -> output:#GND#0
- U$1412, U$1430, U$1451, U$1469, U$632, U$671, U$728, U$767: device output:#GND#0 -> output:#SCLK#0
- U$1414, U$1432, U$634, U$730: device output:#SCLK#0 -> output:#SDA#0
- U$1415, U$1433, U$635, U$731: device output:#COPI#0 -> output:#CIPO#0
- U$1416, U$1434, U$636, U$732: device output:#SDA#0 -> output:#GPIO1#0
- U$1417, U$1435, U$637, U$733: device output:#CIPO#0 -> output:#CS0#0
- U$1418, U$1436, U$638, U$734: device output:#GPIO1#0 -> output:#GPIO0#0
- U$1419, U$1437, U$639, U$735: device output:#CS0#0 -> output:#CS1#0
- U$1420, U$1438, U$640, U$736: device output:#GPIO0#0 -> output:#CS2#0
- U$1421, U$641: device output:#CS1#0 -> output:#I�C#0
- U$1422, U$1478, U$642, U$776: device output:#CS2#0 -> output:#SCL#0
- U$1423, U$625: value (none) -> SPARKX-LOGO3; device output:#I�C#0 -> SparkX:SPARKX-SMALL
- U$1441, U$1479, U$778, U$816: device output:#SCL#0 -> output:SM�L_HEADER0
- U$1442, U$1481: device output:SM�L_HEADER0 -> output:OUT0
- U$1444, U$760: value (none) -> SPARKX-LOGO3; device output:OUT0 -> SparkX:SPARKX-SMALL
- U$1445, U$1463, U$665, U$761: value SPARKX-LOGO3 -> (none); device SparkX:SPARKX-SMALL -> output:#V_USB#0
- U$1452, U$1470, U$672, U$768: device output:#SCLK#0 -> output:#COPI#0
- U$1453, U$1471, U$673, U$769: device output:#COPI#0 -> output:#SDA#0
- U$1454, U$1472, U$674, U$770: device output:#SDA#0 -> output:#CIPO#0
- U$1455, U$1473, U$675, U$771: device output:#CIPO#0 -> output:#GPIO1#0
- U$1456, U$1474, U$676, U$772: device output:#GPIO1#0 -> output:#CS0#0
- U$1457, U$1475, U$677, U$773: device output:#CS0#0 -> output:#GPIO0#0
- U$1458, U$1476, U$678, U$774: device output:#GPIO0#0 -> output:#CS1#0
- U$1459, U$1477, U$679, U$775: device output:#CS1#0 -> output:#CS2#0
- U$1460, U$680: device output:#CS2#0 -> output:#I�C#0
- U$1461, U$815: device output:#I�C#0 -> output:#SCL#0
- U$1482: value (none) -> SMOL_LOGOSMALL; device output:OUT0 -> SparkX:SMOL_SMALL
- U$149, U$1631, U$1652, U$170, U$833, U$968: device output:#SCL#0 -> output:#GPIO0#0
- U$150, U$1632, U$1671, U$189, U$834, U$873: device output:SM�L_HEADER0 -> output:#CS1#0
- U$152, U$1634, U$798: device output:OUT0 -> output:#SCL#0
- U$1521, U$39, U$741: value SPARKX-LOGO3 -> SMOL_LOGOSMALL; device SparkX:SPARKX-SMALL -> SparkX:SMOL_SMALL
- U$1522, U$1540, U$40, U$58, U$742, U$838: value (none) -> SPARKX-LOGO3; device output:#V_USB#0 -> SparkX:SPARKX-SMALL
- U$1523, U$1541, U$1562, U$1580, U$41, U$59, U$743, U$782, U$80, U$839, U$878, U$98: device output:#3#3V#0 -> output:#V_USB#0
- U$1525, U$1543, U$1563, U$1581, U$43, U$61, U$745, U$783, U$81, U$841, U$879, U$99: device output:#PWR_EN#0 -> output:#3#3V#0
- U$1529, U$1547, U$47, U$65, U$749, U$845: device output:#COPI#0 -> output:#SCLK#0
- U$1530, U$1548, U$48, U$66, U$750, U$846: device output:#SDA#0 -> output:#COPI#0
- U$1531, U$1549, U$49, U$67, U$751, U$847: device output:#CIPO#0 -> output:#SDA#0
- U$1532, U$1550, U$50, U$68, U$752, U$848: device output:#GPIO1#0 -> output:#CIPO#0
- U$1533, U$1551, U$51, U$69, U$753, U$849: device output:#CS0#0 -> output:#GPIO1#0
- U$1534, U$1552, U$52, U$70, U$754, U$850: device output:#GPIO0#0 -> output:#CS0#0
- U$1535, U$1553, U$53, U$71, U$755, U$851: device output:#CS1#0 -> output:#GPIO0#0
- U$1536, U$1554, U$54, U$72, U$756, U$852: device output:#CS2#0 -> output:#CS1#0
- U$1537, U$55, U$853: device output:#I�C#0 -> output:#CS2#0
- U$1538, U$56, U$719: device output:#SCL#0 -> output:#I�C#0
- U$1539, U$1673, U$191, U$57, U$837, U$893: value SPARKX-LOGO3 -> (none); device SparkX:SPARKX-SMALL -> output:#SCL#0
- U$154, U$1636, U$1674, U$192, U$856, U$894: device output:#V_USB#0 -> output:SM�L_HEADER0
- U$155, U$1637, U$1676, U$194, U$857, U$896: device output:#3#3V#0 -> output:OUT0
- U$1555, U$1576, U$73, U$757, U$892, U$94: device output:#SCL#0 -> output:#CS2#0
- U$1559, U$77, U$779: value SPARKX-LOGO3 -> (none); device SparkX:SPARKX-SMALL -> output:OUT0
- U$1560, U$78, U$780: value (none) -> SMOL_LOGOSMALL; device output:#V_USB#0 -> SparkX:SMOL_SMALL
- U$157, U$1639, U$1657, U$175, U$859, U$955: value (none) -> SPARKX-LOGO3; device output:#PWR_EN#0 -> SparkX:SPARKX-SMALL
- U$1575, U$891, U$93: device output:#I�C#0 -> output:#CS1#0
- U$1577, U$875, U$95: value SPARKX-LOGO3 -> (none); device SparkX:SPARKX-SMALL -> output:#I�C#0
- U$1578, U$1712, U$230, U$876, U$932, U$96: device output:#V_USB#0 -> output:#SCL#0
- U$158, U$1640, U$1658, U$1679, U$1697, U$176, U$197, U$215, U$860, U$899, U$956, U$995: device output:#GND#0 -> output:#V_USB#0
- U$160, U$1642, U$1660, U$1680, U$1698, U$178, U$198, U$216, U$862, U$900, U$958, U$996: device output:#SCLK#0 -> output:#3#3V#0
- U$161, U$1643, U$1661, U$179, U$863, U$959: device output:#COPI#0 -> output:#PWR_EN#0
- U$163, U$1645, U$1663, U$1683, U$1701, U$181, U$201, U$219, U$865, U$903, U$961, U$999: device output:#CIPO#0 -> output:#GND#0
- U$164, U$1646, U$1664, U$182, U$866, U$962: device output:#GPIO1#0 -> output:#SCLK#0
- U$1647, U$165, U$1665, U$183, U$867, U$963: device output:#CS0#0 -> output:#COPI#0
- U$1648, U$166, U$1666, U$184, U$868, U$964: device output:#GPIO0#0 -> output:#SDA#0
- U$1649, U$1667, U$167, U$185, U$869, U$965: device output:#CS1#0 -> output:#CIPO#0
- U$1650, U$1668, U$168, U$186, U$870, U$966: device output:#CS2#0 -> output:#GPIO1#0
- U$1651, U$169, U$967: device output:#I�C#0 -> output:#CS0#0
- U$1653, U$171, U$1749, U$267, U$951, U$969: value SPARKX-LOGO3 -> (none); device SparkX:SPARKX-SMALL -> output:#CS1#0
- U$1654, U$172, U$1750, U$268, U$952, U$970: device output:#V_USB#0 -> output:#CS2#0
- U$1655, U$1694, U$173, U$212, U$953, U$992: device output:#3#3V#0 -> output:#I�C#0
- U$1670, U$1709, U$188, U$227, U$872, U$911: device output:SM�L_HEADER0 -> output:#GPIO0#0
- U$1672, U$190, U$874: device output:OUT0 -> output:#CS2#0
- U$1675, U$1713, U$1714, U$1752, U$193, U$231, U$232, U$270, U$895, U$933, U$934, U$972: device output:#3#3V#0 -> output:SM�L_HEADER0
- U$1677, U$195, U$897: value (none) -> SMOL_LOGOSMALL; device output:#PWR_EN#0 -> SparkX:SMOL_SMALL
- U$1682, U$1700, U$200, U$218, U$902, U$998: device output:#SDA#0 -> output:#PWR_EN#0
- U$1708, U$1747, U$226, U$265, U$910, U$949: device output:SM�L_HEADER0 -> output:#CS0#0
- U$1710, U$228, U$912: device output:OUT0 -> output:#CS1#0
- U$1715, U$233, U$935: device output:#PWR_EN#0 -> output:OUT0
- U$1716, U$1755, U$234, U$273, U$936, U$975: value (none) -> SMOL_LOGOSMALL; device output:#GND#0 -> SparkX:SMOL_SMALL
- U$1746, U$1785, U$264, U$303, U$948, U$987: device output:SM�L_HEADER0 -> output:#GPIO1#0
- U$1748, U$266, U$950: device output:OUT0 -> output:#GPIO0#0
- U$1786, U$304, U$988: device output:OUT0 -> output:#CS0#0
- U$663: value (none) -> SMOL_LOGOSMALL; device output:#I�C#0 -> SparkX:SMOL_SMALL
- U$701: device output:#I�C#0 -> output:OUT0
- U$739, U$777: device output:#I�C#0 -> output:SM�L_HEADER0
- U$758, U$797: device output:SM�L_HEADER0 -> output:#I�C#0
- U$836: device output:OUT0 -> output:#I�C#0
- moved U$624 181.2 mm to (173.0, 6.92)
- moved U$622 180.3 mm to (173.0, 5.59), flipped to the bottom
- moved U$1248 179.9 mm to (173.0, 48.1), flipped to the top
- moved U$1232 179.7 mm to (173.3, 53.3), flipped to the bottom
- moved U$1246 179.5 mm to (173.0, 46.7)
- moved U$1228 178.8 mm to (173.0, 48.8), flipped to the bottom
- moved U$623 178.8 mm to (173.0, 5.08)
- moved U$1247 177.9 mm to (173.0, 46.2), flipped to the top
- moved U$621 176.8 mm to (173.0, 8.32)
- moved U$1231 176.7 mm to (174.4, 55.9), flipped to the bottom
- moved U$1245 176.1 mm to (173.0, 49.5), flipped to the top
- moved U$1230 175.7 mm to (171.6, 56.8), flipped to the bottom
- moved U$1233 175.4 mm to (174.4, 58.5), flipped to the bottom
- moved U$1226 174.9 mm to (176.0, 74.2)
- moved U$1229 174.4 mm to (172.1, 54.4), flipped to the bottom
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